File: CAD/PCB/r2_0/kicad/PulsePalSMT_Rev_0_5.kicad_pcb (KiCad board)
At the start: 4 copper layers, 99 x 82.6 mm, 53 parts, among them IC1 OPTOISOLATOR-2SOIC8, IC2 AD5754RBREZ, IC3 REG1117, U1 USD-SOCKET, U2 TDK_LAMBDA_5_TO_BI_12_125MA

Commit message: PCB/r2_0/kicad: 2 layer PCB
Signed-off-by: Ilya Kuzmin <kuzmin.ilya@gmail.com>
Parts:
- removed AGND26, DGND26: , 1X01
- removed ARDUINO26: DUE(NORMAL), DUE(NORMAL)
- removed THUMB_CONTROLLER26: , JOYSTICK
- added AGND: , 1X01, F.Cu at (195.2, 121.6)
- added ARDUINO: DUE(NORMAL), DUE(NORMAL), F.Cu at (166.7, 104.0)
- added DGND: , 1X01, F.Cu at (195.1, 116.4)
- added THUMB_CONTROLLER: , JOYSTICK, F.Cu at (186.3, 81.8)
- moved U$6 1.70 mm to (157.5, 115.5)
Connections:
- BNC1 pad SIGN: (no net) -> N$8
- BNC2 pad SIGN: (no net) -> N$10
- BNC3 pad SIGN: (no net) -> N$3
- BNC4 pad SIGN: (no net) -> N$4
- BNC5 pad SIGN: (no net) -> N$5
- BNC6 pad SIGN: (no net) -> N$6
Routing:
- net GND: track 56.4 -> 177.9 mm, vias 16 -> 44
- net AGND: track 13.6 -> 54.0 mm, vias 4 -> 2
- net 5V: track 95.1 -> 99.9 mm
- net N$9: track 19.5 -> 21.3 mm
- net N$6: track 44.2 -> 45.2 mm
- net VCC: track 152.0 -> 152.7 mm
- net N$40: track 45.3 -> 45.6 mm, vias 2 -> 3
- added copper zone on B.Cu, net AGND
- added copper zone on B.Cu, net GND
- removed copper zone on Route2, net AGND
- removed copper zone on Route15, net GND
Other:
- net class Default: trace_width 0.25 -> 1; via_dia 0.8 -> 3; via_drill 0.4 -> 2
